File: Hardware/UartWifiBoard/UartWifiBoard.sch (EAGLE design)
At the start: 39 parts, among them CN1 B2B-XH, CN2 B4B-XH, CN3 B5B-PH, IC1 ESP-WROOM-02, Q1 RN1302, Q2 RN2302, Q3 TLP2368, Q4 TLP2368, Q5 RN2302, SW1 SKRPACE010, SW2 SKRPACE010, U1 NJM2884U1

Commit message: Upload files
Parts:
- removed LED3: OSHR1608C1A, optosupply:OSHR1608C1A
- removed Q5: RN2302, toshiba:RN2302
- removed R3: 220, rcl:R-EU_R0603
- removed R99: 0ohm, rcl:R-EU_R0603
- added C7, C8: 0.1u, rcl:C-EUC0603
- added D1: RB521S30, on-semiconductor:RB521S30
- added OLED1: DISPLAY-OLED-128X32, generic-brand-oled-modules:DISPLAY-OLED-128X32
- added PC1, PC2: TLP2368, toshiba:TLP2368
- added R12: 10.0k, rcl:R-EU_R0603
- added R13: 3.3k, rcl:R-EU_R0603
- added R14: 470, rcl:R-EU_R0603
- added R15: 1.0k, rcl:R-EU_R0603
- added SW3: SKRPACE010, alps:SKRPACE010
- C2, C3: value 1.0u -> 2.2u
- LED1: value OSTG1608C1A -> OSOR1608C1A; device optosupply:OSTG1608C1A -> optosupply:OSOR1608C1A
- LED2: value OSYL1608C1A -> OSHR1608C1A; device optosupply:OSYL1608C1A -> optosupply:OSHR1608C1A
- Q1: value RN1302 -> MMUN2211LT1G; device toshiba:RN1302 -> on-semiconductor:MMUN2211LT1G
- Q2: value RN2302 -> MMUN2111LT1G; device toshiba:RN2302 -> on-semiconductor:MMUN2111LT1G
- Q3: value TLP2368 -> MMUN2211LT1G; device toshiba:TLP2368 -> on-semiconductor:MMUN2211LT1G
- Q4: value TLP2368 -> MMUN2111LT1G; device toshiba:TLP2368 -> on-semiconductor:MMUN2111LT1G
- R10: value 1.0k -> 3.3k
- R11: value 220 -> 3.3k
- R24: value 3.3k -> 4.7k
- R4: value 3.3k -> 220
- R7, R8: value 10.0k -> 3.3k
- R9: value 470 -> 3.3k
Connections:
- removed net N$10: CN3.5, R11.2
- removed net N$18: IC1.IO15, R8.2
- removed net N$9: LED2.A, R4.1
- new net IO12: IC1.IO12, Q3.C, R5.1
- new net IO13: IC1.IO13, R8.1, SW3.1, SW3.2
- new net IO15: IC1.IO15, R11.2
- new net IO16: IC1.IO16, R7.1, SW2.1, SW2.2
- new net IO4: IC1.IO4, OLED1.SDA
- new net IO5: IC1.IO5, OLED1.SCL
- new net N$14: D1.A, Q3.B, SW1.3, SW1.4
- net IO0: now also CN3.5, R9.1; no longer LED1.C, R11.1
- net IO2: now also LED1.C, R10.1; no longer LED2.C
- net N$11: now also PC1.VO; no longer Q3.VO
- net N$13: now also LED2.A; no longer LED3.A
- net N$16: now also PC1.A, R14.1; no longer Q3.A, R9.1
- net N$19: now also R12.1; no longer R7.1
- net N$2: now also R4.2; no longer R3.2
- net N$22: now also R6.1; no longer R5.1
- net N$3: no longer R99.1
- net N$4: now also Q4.C; no longer Q5.C
- net N$5: now also D1.C, R4.1; no longer R3.1, R99.2, SW1.3, SW1.4
- net N$7: now also Q4.B; no longer Q5.B
- net N$8: now also PC2.A; no longer Q4.A
- net P+3V3: now also C8.1, OLED1.VCC, PC2.VCC, R12.2, R13.2, R14.2, R15.2, R8.2; no longer Q4.VCC, R4.2
- net PGND: now also C7.2, C8.2, OLED1.GND, PC2.GND, Q3.E, R11.1, SW3.3, SW3.4; no longer Q4.GND, R8.1
- net RST: now also C7.1, R13.1; no longer R6.1
- net RXD: now also PC2.VO, R15.1; no longer Q4.VO, R10.1
- net S+SUP: now also PC1.VCC, Q4.E; no longer Q3.VCC, Q5.E
- net SGND: now also LED2.C, PC1.GND, PC2.K; no longer LED3.C, Q3.GND, Q4.K
- net TOUT: no longer SW2.1, SW2.2
- net TXD: now also PC1.K; no longer Q3.K
Other:
- note removed: "02"
